Commit message: chore: auto-sync 2026-10-07 23:00

File: my_robot_description/urdf/my_robot.urdf (robot description, URDF)
Before this commit: robot swan_drone, 1 links, 0 joints
Links:
- added link right_wheel_link; visual cylinder length=0.05 radius=0.1
- link base_link: geometry visual box size=0.6 0.4 0.2
Joints:
- added joint base_right_wheel_joint: type fixed, parent base_link, child right_wheel_link, origin xyz=0 0 0 rpy=0 0 0

Commit message: feat(my_robot_description): implement modular Xacro URDF, macros, and RViz launch file

File: my_robot_description/urdf/my_robot.urdf (robot description, URDF)
Before this commit: robot my_robot, 2 links, 1 joints
Links:
- added link base_footprint
- added link caster_wheel_link; visual sphere radius=0.05
- added link left_wheel_link; visual cylinder length=0.05 radius=0.1
Joints:
- added joint base_caster_wheel_joint: type fixed, parent base_link, child caster_wheel_link, origin xyz=0.2 0 -0.05 rpy=0 0 0
- added joint base_joint: type fixed, parent base_footprint, child base_link, origin xyz=0 0 0.1 rpy=0 0 0
- added joint base_left_wheel_joint: type continuous, parent base_link, child left_wheel_link, origin xyz=-0.15 0.225 0 rpy=0 0 0, axis 0 1 0
- joint base_right_wheel_joint: axis (none) -> 0 1 0; origin xyz=0 0 0 rpy=0 0 0 -> xyz=-0.15 -0.225 0 rpy=0 0 0; type fixed -> continuous
